Commit message: Add Lidar pluggin for Gazebo and Rviz
Data from lidar can be visualise inside Gazebo and Rviz. Some changes can be done on the display of the ray in Gazebo (color and size).
New config file has been added to open Rviz with the correct topic.
Minor correction: camera's orientation is rectified.

File: src/billy_description/urdf/billy_v0.xacro (robot description, xacro)
@@ -210,5 +210,5 @@
     </gazebo>
     <joint name="cam_joint" type="fixed">
-      <origin xyz="0.112 0 0.053" rpy="1.57 0 1.57" />
+      <origin xyz="0.112 0 0.053" rpy="0 0 0" />
       <parent link="base_link"/>
       <child link="cam_link" />
@@ -219,5 +219,5 @@
          <mesh scale="0.001 0.001 0.001" filename="package://billy_description/meshes/TurtlebotBilly_SheldCam.stl"/>
         </geometry>
-        <origin xyz="0 0 0" rpy="0 0 0"/>
+        <origin xyz="0 0 0" rpy="1.57 0 1.57" />
       </visual>
       <collision>
@@ -225,5 +225,5 @@
          <mesh scale="0.001 0.001 0.001" filename="package://billy_description/meshes/TurtlebotBilly_SheldCam.stl"/>
         </geometry>
-        <origin xyz="0 0 0.0" rpy="0 0 0"/>
+        <origin xyz="0 0 0" rpy="1.57 0 1.57" />
       </collision>
     </link>
@@ -486,5 +486,35 @@
         <distortionT2>0.0</distortionT2>
       </plugin>
-    </sensor>
-  </gazebo>
+      </sensor>
+    </gazebo>
+    <gazebo reference="lidar_link"><sensor type="gpu_ray" name="head_rplidar_sensor">
+        <!--pose>0 0 0 0 0 0</pose -->
+        <visualize>true</visualize>
+        <update_rate>10</update_rate>
+        <ray>
+          <scan>
+            <horizontal>
+              <samples>400</samples>
+              <resolution>1</resolution>
+              <min_angle>-3.14159</min_angle>
+              <max_angle>3.14159</max_angle>
+            </horizontal>
+          </scan>
+          <range>
+            <min>0.15</min>
+            <max>6.0</max>
+            <resolution>0.01</resolution>
+          </range>
+          <noise>
+            <type>gaussian</type>
+            <mean>0.0</mean>
+            <stddev>0.01</stddev>
+          </noise>
+        </ray>
+        <plugin name="gazebo_ros_head_rplidar_controller" filename="libgazebo_ros_gpu_laser.so">
+          <topicName>/scan</topicName>
+          <frameName>lidar_link</frameName>
+        </plugin>
+      </sensor>
+    </gazebo>
 </robot>

Commit message: Add Lidar and camera support for real robot
Changed rplidar.launch file to USB1 before and "standard" mode. Added a "laser" link inside the .xacro file.
Added usb_cam node and rplidar.launch inside rosserial rasp launch file.
Minor changes to config of Rviz when opening

File: src/billy_description/urdf/billy_v0.xacro (robot description, xacro)
@@ -209,4 +209,10 @@
       <material>Gazebo/DarkGrey</material>
     </gazebo>
+    <joint name="laser_joint" type="fixed">
+      <origin xyz="0 0 0" rpy="0 0 0" />
+      <parent link="lidar_link"/>
+      <child link="laser" />
+    </joint>
+    <link name="laser"></link>
     <joint name="cam_joint" type="fixed">
       <origin xyz="0.112 0 0.053" rpy="0 0 0" />

Commit message: Enhancement of .xacro with update of the corresponding parent link
.xacro of billy use to have all parent link set as "base_link". This has been change to true parent of the component (matching with real life). Makes it easier to update component after.
base_footprint has been added to naviguation purposes.
Good practices has been delete replaced by the README.md in the rosserial package

File: src/billy_description/urdf/billy_v0.xacro (robot description, xacro)
@@ -2,5 +2,4 @@
 <robot name="billy_v2" xmlns:xacro="http://www.ros.org/wiki/xacro">
     <!-- Joint, link and color of components -->
-    <!--
     <link name="base_footprint"/>
     <joint name="base_joint" type="fixed">
@@ -9,5 +8,4 @@
       <child link="base_link"/>
     </joint>
-    -->
     <link name="base_link">
       <visual>
@@ -34,10 +32,112 @@
       <material>Gazebo/White</material>
     </gazebo>
+    <joint name="stand_1_joint" type="fixed">
+      <origin xyz="0.108 0.108 -0.005" rpy="0 0 0" />
+      <parent link="base_link"/>
+      <child link="stand_1_link" />
+    </joint>
+    <link name="stand_1_link">
+      <visual>
+        <geometry>
+         <mesh scale="0.001 0.001 0.001" filename="package://billy_description/meshes/VisM6x40.stl"/>
+        </geometry>
+        <origin xyz="0 0 0" rpy="0 0 0" />
+      </visual>
+      <collision>
+        <geometry>
+         <mesh scale="0.001 0.001 0.001" filename="package://billy_description/meshes/VisM6x40.stl"/>
+        </geometry>
+        <origin xyz="0 0 0" rpy="0 0 0" />
+      </collision>
+      <!--inertial>
+        <origin xyz="0.0 0 0"/>
+        <mass value="1.0"/>
+        <inertia ixx="0.019995" ixy="0.0" ixz="0.0"
+                 iyy="0.019995" iyz="0.0"
+                 izz="0.03675" />
+      </inertial-->
+    </link>
+    <gazebo reference="stand_1_link">
+      <material>Gazebo/Grey</material>
+    </gazebo>
+    <joint name="stand_2_joint" type="fixed">
+      <origin xyz="-0.108 0.108 -0.005" rpy="0 0 0" />
+      <parent link="base_link"/>
+      <child link="stand_2_link" />
+    </joint>
+    <link name="stand_2_link">
+      <visual>
+        <geometry>
+         <mesh scale="0.001 0.001 0.001" filename="package://billy_description/meshes/VisM6x40.stl"/>
+        </geometry>
+        <origin xyz="0 0 0" rpy="0 0 0" />
+      </visual>
+      <collision>
+        <geometry>
+         <mesh scale="0.001 0.001 0.001" filename="package://billy_description/meshes/VisM6x40.stl"/>
+        </geometry>
+        <origin xyz="0 0 0" rpy="0 0 0" />
+      </collision>
+      <!--inertial>
+        <origin xyz="0.0 0 0"/>
+        <mass value="1.0"/>
+        <inertia ixx="0.019995" ixy="0.0" ixz="0.0"
+                 iyy="0.019995" iyz="0.0"
+                 izz="0.03675" />
+      </inertial-->
+    </link>
+    <gazebo reference="stand_2_link">
+      <material>Gazebo/Grey</material>
+    </gazebo>
+    <joint name="stand_3_joint" type="fixed">
+      <origin xyz="-0.108 -0.108 -0.005" rpy="0 0 0" />
+      <parent link="base_link"/>
+      <child link="stand_3_link" />
+    </joint>
+    <link name="stand_3_link">
+      <visual>
+        <geometry>
+         <mesh scale="0.001 0.001 0.001" filename="package://billy_description/meshes/VisM6x40.stl"/>
+        </geometry>
+        <origin rpy="0 0 0" xyz="0 0 0.0"/>
+      </visual>
+      <collision>
+        <geometry>
+         <mesh scale="0.001 0.001 0.001" filename="package://billy_description/meshes/VisM6x40.stl"/>
+        </geometry>
+        <origin rpy="0 0 0" xyz="0 0 0.0"/>
+      </collision>
+    </link>
+    <gazebo reference="stand_3_link">
+      <material>Gazebo/Grey</material>
+    </gazebo>
+    <joint name="stand_4_joint" type="fixed">
+      <origin xyz="0.108 -0.108 -0.005" rpy="0 0 0" />
+      <parent link="base_link"/>
+      <child link="stand_4_link" />
+    </joint>
+    <link name="stand_4_link">
+      <visual>
+        <geometry>
+         <mesh scale="0.001 0.001 0.001" filename="package://billy_description/meshes/VisM6x40.stl"/>
+        </geometry>
+        <origin rpy="0 0 0" xyz="0 0 0.0"/>
+      </visual>
+      <collision>
+        <geometry>
+         <mesh scale="0.001 0.001 0.001" filename="package://billy_description/meshes/VisM6x40.stl"/>
+        </geometry>
+        <origin rpy="0 0 0" xyz="0 0 0.0"/>
+      </collision>
+    </link>
+    <gazebo reference="stand_4_link">
+      <material>Gazebo/Grey</material>
+    </gazebo>
     <joint name="second_level_joint" type="fixed">
-      <origin xyz="0 0 0.03" rpy="0 0 0" />
-      <parent link="base_link"/>
-      <child link="base_second_link"/>
-    </joint>
-    <link name="base_second_link">
+      <origin xyz="-0.108 -0.108 0.035" rpy="0 0 0" />
+      <parent link="stand_1_link"/>
+      <child link="second_level_link"/>
+    </joint>
+    <link name="second_level_link">
       <visual>
         <geometry>
@@ -63,109 +163,7 @@
       <material>Gazebo/White</material>
     </gazebo>
-    <joint name="stand_1_joint" type="fixed">
-      <origin xyz="0.108 0.108 -0.005" rpy="0 0 0" />
-      <parent link="base_link"/>
-      <child link="stand_1_link" />
-    </joint>
-    <link name="stand_1_link">
-      <visual>
-        <geometry>
-         <mesh scale="0.001 0.001 0.001" filename="package://billy_description/meshes/VisM6x40.stl"/>
-        </geometry>
-        <origin xyz="0 0 0" rpy="0 0 0" />
-      </visual>
-      <collision>
-        <geometry>
-         <mesh scale="0.001 0.001 0.001" filename="package://billy_description/meshes/VisM6x40.stl"/>
-        </geometry>
-        <origin xyz="0 0 0" rpy="0 0 0" />
-      </collision>
-      <!--inertial>
-        <origin xyz="0.0 0 0"/>
-        <mass value="1.0"/>
-        <inertia ixx="0.019995" ixy="0.0" ixz="0.0"
-                 iyy="0.019995" iyz="0.0"
-                 izz="0.03675" />
-      </inertial-->
-    </link>
-    <gazebo reference="stand_1_link">
-      <material>Gazebo/Grey</material>
-    </gazebo>
-    <joint name="stand_2_joint" type="fixed">
-      <origin xyz="-0.108 0.108 -0.005" rpy="0 0 0" />
-      <parent link="base_link"/>
-      <child link="stand_2_link" />
-    </joint>
-    <link name="stand_2_link">
-      <visual>
-        <geometry>
-         <mesh scale="0.001 0.001 0.001" filename="package://billy_description/meshes/VisM6x40.stl"/>
-        </geometry>
-        <origin xyz="0 0 0" rpy="0 0 0" />
-      </visual>
-      <collision>
-        <geometry>
-         <mesh scale="0.001 0.001 0.001" filename="package://billy_description/meshes/VisM6x40.stl"/>
-        </geometry>
-        <origin xyz="0 0 0" rpy="0 0 0" />
-      </collision>
-      <!--inertial>
-        <origin xyz="0.0 0 0"/>
-        <mass value="1.0"/>
-        <inertia ixx="0.019995" ixy="0.0" ixz="0.0"
-                 iyy="0.019995" iyz="0.0"
-                 izz="0.03675" />
-      </inertial-->
-    </link>
-    <gazebo reference="stand_2_link">
-      <material>Gazebo/Grey</material>
-    </gazebo>
-    <joint name="stand_3_joint" type="fixed">
-      <origin xyz="-0.108 -0.108 -0.005" rpy="0 0 0" />
-      <parent link="base_link"/>
-      <child link="stand_3_link" />
-    </joint>
-    <link name="stand_3_link">
-      <visual>
-        <geometry>
-         <mesh scale="0.001 0.001 0.001" filename="package://billy_description/meshes/VisM6x40.stl"/>
-        </geometry>
-        <origin rpy="0 0 0" xyz="0 0 0.0"/>
-      </visual>
-      <collision>
-        <geometry>
-         <mesh scale="0.001 0.001 0.001" filename="package://billy_description/meshes/VisM6x40.stl"/>
-        </geometry>
-        <origin rpy="0 0 0" xyz="0 0 0.0"/>
-      </collision>
-    </link>
-    <gazebo reference="stand_3_link">
-      <material>Gazebo/Grey</material>
-    </gazebo>
-    <joint name="stand_4_joint" type="fixed">
-      <origin xyz="0.108 -0.108 -0.005" rpy="0 0 0" />
-      <parent link="base_link"/>
-      <child link="stand_4_link" />
-    </joint>
-    <link name="stand_4_link">
-      <visual>
-        <geometry>
-         <mesh scale="0.001 0.001 0.001" filename="package://billy_description/meshes/VisM6x40.stl"/>
-        </geometry>
-        <origin rpy="0 0 0" xyz="0 0 0.0"/>
-      </visual>
-      <collision>
-        <geometry>
-         <mesh scale="0.001 0.001 0.001" filename="package://billy_description/meshes/VisM6x40.stl"/>
-        </geometry>
-        <origin rpy="0 0 0" xyz="0 0 0.0"/>
-      </collision>
-    </link>
-    <gazebo reference="stand_4_link">
-      <material>Gazebo/Grey</material>
-    </gazebo>
     <joint name="lidar_shield_joint" type="fixed">
-      <origin xyz="0 0 0.04" rpy="0 0 0" />
-      <parent link="base_link"/>
+      <origin xyz="0 0 0.01" rpy="0 0 0" />
+      <parent link="second_level_link"/>
       <child link="lidar_shield_link" />
     </joint>
@@ -188,6 +186,6 @@
     </gazebo>
     <joint name="lidar_joint" type="fixed">
-      <origin xyz="0 0 0.065" rpy="0 0 1.57" />
-      <parent link="base_link"/>
+      <origin xyz="0 0 0.028" rpy="0 0 1.57" />
+      <parent link="lidar_shield_link"/>
       <child link="lidar_link" />
     </joint>
@@ -216,6 +214,6 @@
     <link name="laser"></link>
     <joint name="cam_joint" type="fixed">
-      <origin xyz="0.112 0 0.053" rpy="0 0 0" />
-      <parent link="base_link"/>
+      <origin xyz="0.112 0 0.023" rpy="0 0 0" />
+      <parent link="second_level_link"/>
       <child link="cam_link" />
     </joint>
@@ -260,7 +258,7 @@
     </gazebo>
     <joint name="front_wheel_joint" type="fixed">
-      <parent link="base_link"/>
+      <parent link="front_wheel_holder_link"/>
       <child link="front_wheel_link"/>
-      <origin xyz="0.07 0 -0.035" rpy="1.57 0 0"/>
+      <origin xyz="0 0 -0.028" rpy="1.57 0 0"/>
     </joint>
     <link name="front_wheel_link">
@@ -290,7 +288,29 @@
       <material>Gazebo/Orange</material>
     </gazebo>
+    <joint name="wheel_left_holder_joint" type="fixed">
+      <origin xyz="-0.118 -0.129 -0.023" rpy="0 0 0" />
+      <parent link="base_link"/>
+      <child link="wheel_left_holder_link" />
+    </joint>
+    <link name="wheel_left_holder_link">
+      <visual>
+        <geometry>
+         <mesh scale="0.001 0.001 0.001" filename="package://billy_description/meshes/TurtlebotBilly_Motor_ShieldL_v1.stl"/>
+        </geometry>
+        <origin xyz="0 0 0" rpy="0 0 0"/>
+      </visual>
+      <collision>
+        <geometry>
+         <mesh scale="0.001 0.001 0.001" filename="package://billy_description/meshes/TurtlebotBilly_Motor_ShieldL_v1.stl"/>
+        </geometry>
+        <origin xyz="0 0 0.0" rpy="0 0 0"/>
+      </collision>
+    </link>
+    <gazebo reference="wheel_left_holder_link">
+      <material>Gazebo/Orange</material>
+    </gazebo>
     <joint name="motor_left_joint" type="fixed">
-      <origin xyz="-0.080 -0.125 -0.023" rpy="0 0 0" />
-      <parent link="base_link"/>
+      <origin xyz="0.038 0.004 0" rpy="0 0 0" />
+      <parent link="wheel_left_holder_link"/>
       <child link="motor_left_link" />
     </joint>
@@ -313,30 +333,8 @@
       <material>Gazebo/Grey</material>
     </gazebo>
-    <joint name="wheel_left_holder_joint" type="fixed">
-      <origin xyz="-0.118 -0.129 -0.023" rpy="0 0 0" />
-      <parent link="base_link"/>
-      <child link="wheel_left_holder_link" />
-    </joint>
-    <link name="wheel_left_holder_link">
-      <visual>
-        <geometry>
-         <mesh scale="0.001 0.001 0.001" filename="package://billy_description/meshes/TurtlebotBilly_Motor_ShieldL_v1.stl"/>
-        </geometry>
-        <origin xyz="0 0 0" rpy="0 0 0"/>
-      </visual>
-      <collision>
-        <geometry>
-         <mesh scale="0.001 0.001 0.001" filename="package://billy_description/meshes/TurtlebotBilly_Motor_ShieldL_v1.stl"/>
-        </geometry>
-        <origin xyz="0 0 0.0" rpy="0 0 0"/>
-      </collision>
-    </link>
-    <gazebo reference="wheel_left_holder_link">
-      <material>Gazebo/Orange</material>
-    </gazebo>
     <joint name="wheel_left_joint" type="continuous">
-      <parent link="base_link"/>
+      <parent link="motor_left_link"/>
       <child link="wheel_left_link"/>
-      <origin xyz="-0.075 -0.150 -0.03" rpy="-1.57 0 0"/>
+      <origin xyz="0 -0.022 0" rpy="-1.57 0 0"/>
       <axis xyz="0 0 1"/>
     </joint>
@@ -366,7 +364,30 @@
       <material>Gazebo/Black</material>
     </gazebo>
+    <joint name="wheel_right_holder_joint" type="fixed">
+      <origin xyz="-0.080 0.129 -0.023" rpy="0 0 3.14" />
+      <parent link="base_link"/>
+      <child link="wheel_right_holder_link" />
+    </joint>
+    <link name="wheel_right_holder_link">
+      <color name="yellow" />
+      <visual>
+        <geometry>
+         <mesh scale="0.001 0.001 0.001" filename="package://billy_description/meshes/TurtlebotBilly_Motor_ShieldR_v1.stl"/>
+        </geometry>
+        <origin xyz="0 0 0" rpy="0 0 0"/>
+      </visual>
+      <collision>
+        <geometry>
+         <mesh scale="0.001 0.001 0.001" filename="package://billy_description/meshes/TurtlebotBilly_Motor_ShieldR_v1.stl"/>
+        </geometry>
+        <origin xyz="0 0 0.0" rpy="0 0 0"/>
+      </collision>
+    </link>
+    <gazebo reference="wheel_right_holder_link">
+      <material>Gazebo/Orange</material>
+    </gazebo>
     <joint name="motor_right_joint" type="fixed">
-      <origin xyz="-0.080 0.125 -0.023" rpy="0 3.14 3.14" />
-      <parent link="base_link"/>
+      <origin xyz="0 0.004 0" rpy="0 3.14 0" />
+      <parent link="wheel_right_holder_link"/>
       <child link="motor_right_link" />
     </joint>
@@ -389,31 +410,8 @@
       <material>Gazebo/Grey</material>
     </gazebo>
-    <joint name="wheel_right_holder_joint" type="fixed">
-      <origin xyz="-0.080 0.129 -0.023" rpy="0 0 3.14" />
-      <parent link="base_link"/>
-      <child link="wheel_right_holder_link" />
-    </joint>
-    <link name="wheel_right_holder_link">
-      <color name="yellow" />
-      <visual>
-        <geometry>
-         <mesh scale="0.001 0.001 0.001" filename="package://billy_description/meshes/TurtlebotBilly_Motor_ShieldR_v1.stl"/>
-        </geometry>
-        <origin xyz="0 0 0" rpy="0 0 0"/>
-      </visual>
-      <collision>
-        <geometry>
-         <mesh scale="0.001 0.001 0.001" filename="package://billy_description/meshes/TurtlebotBilly_Motor_ShieldR_v1.stl"/>
-        </geometry>
-        <origin xyz="0 0 0.0" rpy="0 0 0"/>
-      </collision>
-    </link>
-    <gazebo reference="wheel_right_holder_link">
-      <material>Gazebo/Orange</material>
-    </gazebo>
     <joint name="wheel_right_joint" type="continuous">
-      <parent link="base_link"/>
+      <parent link="motor_right_link"/>
       <child link="wheel_right_link"/>
-      <origin xyz="-0.075 0.150 -0.03" rpy="-1.57 0 0"/>
+      <origin xyz="0 -0.023 0" rpy="-1.57 0 0"/>
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
Commit message: Fix bug on xacro file + billy_navigation.launch added
Bug gazebo wheel continuous.
First try to launch navigation with the use of the turtlebot3_navigation package

File: src/billy_description/urdf/billy_v0.xacro (robot description, xacro)
@@ -333,5 +333,5 @@
       <material>Gazebo/Grey</material>
     </gazebo>
-    <joint name="wheel_left_joint" type="continuous">
+    <joint name="wheel_left_joint" type="fixed">
       <parent link="motor_left_link"/>
       <child link="wheel_left_link"/>
@@ -410,5 +410,5 @@
       <material>Gazebo/Grey</material>
     </gazebo>
-    <joint name="wheel_right_joint" type="continuous">
+    <joint name="wheel_right_joint" type="fixed">
       <parent link="motor_right_link"/>
       <child link="wheel_right_link"/>

Commit message: .xacro is update to connect odom to base_footprint
Map is now displaying Rviz while launching billy_navigation.
Need to add map on Rviz and save config

File: src/billy_description/urdf/billy_v0.xacro (robot description, xacro)
@@ -7,4 +7,10 @@
       <parent link="base_footprint"/>
       <child link="base_link"/>
+    </joint>
+    <link name="odom"/>
+    <joint name="odom_joint" type="fixed">
+      <origin xyz="0 0 0" rpy="0 0 0" />
+      <parent link="odom"/>
+      <child link="base_footprint"/>
     </joint>
     <link name="base_link">
