Commit message: Start of the billy_navigation package
Gmmaping is working and amcl as well. Porblem with move_base to be solved

File: src/billy_description/urdf/billy_gazebo.xacro (robot description, xacro)
@@ -450,4 +450,5 @@
         <legacyMode>false</legacyMode>
         <alwaysOn>true</alwaysOn>
+        <rosDebugLevel>na</rosDebugLevel>
         <publishWheelTF>true</publishWheelTF>
         <publishTf>1</publishTf>
@@ -460,8 +461,10 @@
         <wheelAcceleration>1.0</wheelAcceleration>
         <torque>20</torque>
+        <wheelTorque>5</wheelTorque>
         <commandTopic>/cmd_vel</commandTopic>
         <odometryTopic>odom</odometryTopic>
         <odometryFrame>odom</odometryFrame>
-        <robotBaseFrame>base_link</robotBaseFrame>
+        <publishOdomTF>true</publishOdomTF>
+        <robotBaseFrame>base_footprint</robotBaseFrame>
         <odometrySource>world</odometrySource> <!-- 'encoder' instead of 'world' is also possible -->
         <publishTf>1</publishTf>

File: src/billy_description/urdf/billy_rviz.xacro (robot description, xacro)
@@ -340,5 +340,5 @@
     </gazebo>
     <joint name="wheel_left_joint" type="continuous">
-      <parent link="motor_left_link"/>
+      <parent link="odom"/>
       <child link="wheel_left_link"/>
       <origin xyz="0 -0.022 0" rpy="-1.57 0 0"/>
@@ -417,5 +417,5 @@
     </gazebo>
     <joint name="wheel_right_joint" type="continuous">
-      <parent link="motor_right_link"/>
+      <parent link="odom"/>
       <child link="wheel_right_link"/>
       <origin xyz="0 -0.023 0" rpy="-1.57 0 0"/>
