Commit message: Change position of camarm
Switch the shield from second to first stage

File: src/billy_description/urdf/billy_camarm.xacro (robot description, xacro)
@@ -220,5 +220,5 @@
     <link name="laser"></link>
     <joint name="camarm_shield_joint" type="fixed">
-      <origin xyz="0.12 -0.005 0" rpy="0 0 0" />
+      <origin xyz="0.12 -0.005 -0.028" rpy="0 0 0" />
       <parent link="second_level_link"/>
       <child link="camarm_shield_link" />
