Commit message: Modification number of joints
Mismatch number of joint modifications, urdf, launch joint files

File: src/billy_arm/config/billy_links_joints.xacro (robot description, xacro)
@@ -31,25 +31,4 @@
     </joint>
   </xacro:macro>
-<xacro:macro name="m_link_cylinder" params="name origin_xyz origin_rpy radius length mass ixx ixy ixz iyy iyz izz">
-    <link name="${name}">
-      <inertial>
-        <mass value="${mass}" />
-        <origin rpy="${origin_rpy}" xyz="${origin_xyz}" />
-        <inertia ixx="${ixx}" ixy="${ixy}" ixz="${ixz}" iyy="${iyy}" iyz="${iyz}" izz="${izz}" />
-      </inertial>
-      <collision>
-        <origin rpy="${origin_rpy}" xyz="${origin_xyz}" />
-        <geometry>
-          <cylinder radius="${radius}" length="${length}" />
-        </geometry>
-      </collision>
-      <visual>
-        <origin rpy="${origin_rpy}" xyz="${origin_xyz}" />
-        <geometry>
-          <cylinder radius="${radius}" length="${length}" />
-        </geometry>
-      </visual>
-    </link>
-  </xacro:macro>
   <!--<xacro:macro name="m_link_cylinder" params="name origin_xyz origin_rpy radius length mass ixx ixy ixz iyy iyz izz">
     <link name="${name}">

File: src/billy_arm/config/robot_param.xacro (robot description, xacro)
@@ -8,4 +8,3 @@
   <xacro:property name="l05" value="robot_arm_link5" />
   <xacro:property name="l06" value="robot_arm_link6" />
-  <xacro:property name="l07" value="robot_arm_link7" />
 </robot>

File: src/billy_description/urdf/billy_arm.xacro (robot description, xacro)
@@ -279,15 +279,15 @@
             origin_rpy="0 0 0 " origin_xyz="-0.150 0 0"
             scale_xyz="0.01 0.01 0.01"  pathfile="package://billy_description/meshes/Link1.stl"/>
-    <m_joint name="${l02}__${l04}" type="revolute"
+    <m_joint name="${l02}__${l03}" type="revolute"
            axis_xyz="1 0 0"
            limit_e="100" limit_l="-3.14" limit_u="3.14" limit_v="0.25"
            origin_rpy="1.5708 -1.5708 1.5708" origin_xyz="-0.15 0 0.002"
-           parent="${l02}" child="${l04}"/>
-    <transmission name="trans_${l02}__${l04}">
+           parent="${l02}" child="${l03}"/>
+    <transmission name="trans_${l02}__${l03}">
       <type>transmission_interface/SimpleTransmission</type>
-      <joint name="${l02}__${l04}">
+      <joint name="${l02}__${l03}">
         <hardwareInterface>hardware_interface/EffortJointInterface</hardwareInterface>
       </joint>
-      <actuator name="motor_${l02}__${l04}">
+      <actuator name="motor_${l02}__${l03}">
         <hardwareInterface>hardware_interface/EffortJointInterface</hardwareInterface>*
         <mechanicalReduction>1</mechanicalReduction>
@@ -316,5 +316,5 @@
       </actuator>
     </transmission>-->
-    <m_link name="${l04}"
+    <m_link name="${l03}"
             mass="0.5"
             ixx="0.2679" ixy="0.0" ixz="0.0"
@@ -323,8 +323,30 @@
             origin_rpy="0 0 0" origin_xyz="-0.0002 -0.02 -0.07"
             scale_xyz="0.01 0.01 0.01"  pathfile="package://billy_description/meshes/Link3_section_1.stl"/>
+    <m_joint name="${l03}__${l04}" type="revolute"
+           axis_xyz="0 0 1"
+           limit_e="100" limit_l="-3.14" limit_u="3.14" limit_v="0.25"
+           origin_rpy="0 0 0" origin_xyz="0 -0.005 -0.075"
+           parent="${l03}" child="${l04}"/>
+   <transmission name="trans_${l03}__${l04}">
+      <type>transmission_interface/SimpleTransmission</type>
+      <joint name="${l03}__${l04}">
+        <hardwareInterface>hardware_interface/EffortJointInterface</hardwareInterface>
+      </joint>
+      <actuator name="motor_${l03}__${l04}">
+        <hardwareInterface>hardware_interface/EffortJointInterface</hardwareInterface>*
+        <mechanicalReduction>1</mechanicalReduction>
+      </actuator>
+    </transmission>
+    <m_link name="${l04}"
+            mass="0.5"
+            ixx="0.2679" ixy="0.0" ixz="0.0"
+            iyy="0.2679" iyz="0.0"
+            izz="0.0651"
+            origin_rpy="0 0 0" origin_xyz="0.005 0 -0.005"
+            scale_xyz="0.01 0.01 0.01"  pathfile="package://billy_description/meshes/Link3_section_2.stl"/>
     <m_joint name="${l04}__${l05}" type="revolute"
            axis_xyz="0 0 1"
            limit_e="100" limit_l="-3.14" limit_u="3.14" limit_v="0.25"
-           origin_rpy="0 0 0" origin_xyz="0 -0.005 -0.075"
+           origin_rpy="0 1.5708 0" origin_xyz="0 0 -0.04"
            parent="${l04}" child="${l05}"/>
    <transmission name="trans_${l04}__${l05}">
@@ -343,10 +365,26 @@
             iyy="0.2679" iyz="0.0"
             izz="0.0651"
-            origin_rpy="0 0 0" origin_xyz="0.005 0 -0.005"
-            scale_xyz="0.01 0.01 0.01"  pathfile="package://billy_description/meshes/Link3_section_2.stl"/>
+            origin_rpy="0 0 0" origin_xyz="0 0 0.005"
+            scale_xyz="0.01 0.01 0.01"  pathfile="package://billy_description/meshes/Link3_section_3.stl"/>
+    <gazebo reference="${l05}">
+        <mu1>1000</mu1>
+        <mu2>1000</mu2>
+      <kp>1000000.0</kp>
+      <kd>100000.0</kd>
+      <slip1>0</slip1>
+      <slip2>0</slip2>
+      <minDepth>0.001</minDepth>
+      <maxVel>0</maxVel>
+      <torsional>
+          <ode>
+              <coefficient>1000</coefficient>
+              <slip>0</slip>
+          </ode>
+      </torsional>
+    </gazebo>
     <m_joint name="${l05}__${l06}" type="revolute"
            axis_xyz="0 0 1"
            limit_e="100" limit_l="-3.14" limit_u="3.14" limit_v="0.25"
-           origin_rpy="0 1.5708 0" origin_xyz="0 0 -0.04"
+           origin_rpy="3.1416 0 1.5708" origin_xyz="0.0275 0 0.012"
            parent="${l05}" child="${l06}"/>
    <transmission name="trans_${l05}__${l06}">
@@ -365,45 +403,7 @@
             iyy="0.2679" iyz="0.0"
             izz="0.0651"
-            origin_rpy="0 0 0" origin_xyz="0 0 0.005"
-            scale_xyz="0.01 0.01 0.01"  pathfile="package://billy_description/meshes/Link3_section_3.stl"/>
-    <gazebo reference="${l06}">
-        <mu1>1000</mu1>
-        <mu2>1000</mu2>
-      <kp>1000000.0</kp>
-      <kd>100000.0</kd>
-      <slip1>0</slip1>
-      <slip2>0</slip2>
-      <minDepth>0.001</minDepth>
-      <maxVel>0</maxVel>
-      <torsional>
-          <ode>
-              <coefficient>1000</coefficient>
-              <slip>0</slip>
-          </ode>
-      </torsional>
-    </gazebo>
-    <m_joint name="${l06}__${l07}" type="revolute"
-           axis_xyz="0 0 1"
-           limit_e="100" limit_l="-3.14" limit_u="3.14" limit_v="0.25"
-           origin_rpy="3.1416 0 1.5708" origin_xyz="0.0275 0 0.012"
-           parent="${l06}" child="${l07}"/>
-   <transmission name="trans_${l06}__${l07}">
-      <type>transmission_interface/SimpleTransmission</type>
-      <joint name="${l06}__${l07}">
-        <hardwareInterface>hardware_interface/EffortJointInterface</hardwareInterface>
-      </joint>
-      <actuator name="motor_${l06}__${l07}">
-        <hardwareInterface>hardware_interface/EffortJointInterface</hardwareInterface>*
-        <mechanicalReduction>1</mechanicalReduction>
-      </actuator>
-    </transmission>
-    <m_link name="${l07}"
-            mass="0.5"
-            ixx="0.2679" ixy="0.0" ixz="0.0"
-            iyy="0.2679" iyz="0.0"
-            izz="0.0651"
             origin_rpy="0 0 0" origin_xyz="0 0 0"
             scale_xyz="0.01 0.01 0.01"  pathfile="package://billy_description/meshes/End_Effector_Top_Jaw.stl"/>
-    <gazebo reference="${l07}">
+    <gazebo reference="${l06}">
         <mu1>1000</mu1>
         <mu2>1000</mu2>
